Commit message: fix: replace depthimage_to_laserscan with custom node, fix TF tree - Add custom depth_to_scan_node.py that subscribes directly to depth   image topics with matching QoS (RELIABLE/TRANSIENT_LOCAL for images,   RELIABLE/VOLATILE for camera_info), bypassing an image_transport bug   that caused depthimage_to_laserscan to receive 0-height images - Remove base_footprint from URDF to fix disconnected TF trees (both   EKF and URDF were parenting base_link, creating two separate trees) - Disable depth post-processing filters and reduce depth resolution to   480x270x30 to work around RealSense depth stream start failure on   Jetson Orin - Update slam.launch.py depth remappings to use aligned_depth_to_color - Add Transport Hint: raw to RViz depth image display - Register depth_to_scan_node in setup.py entry points

File: urdf/sensor_frames.urdf.xacro (robot description, xacro)
@@ -33,8 +33,6 @@
   <!-- Links                                                               -->
   <!-- ═══════════════════════════════════════════════════════════════════ -->
-  <!-- Base link (provided by platform-specific node or this default) -->
+  <!-- Base link (provided by EKF: odom → base_link) -->
   <link name="base_link"/>
-  <!-- Base footprint (ground plane projection) -->
-  <link name="base_footprint"/>
   <!-- Camera link (D435i body frame) -->
   <link name="camera_link"/>
@@ -44,10 +42,4 @@
   <!-- Joints (static transforms)                                         -->
   <!-- ═══════════════════════════════════════════════════════════════════ -->
-  <!-- base_footprint → base_link (ground to robot center) -->
-  <joint name="base_footprint_to_base" type="fixed">
-    <parent link="base_footprint"/>
-    <child  link="base_link"/>
-    <origin xyz="0 0 0.05" rpy="0 0 0"/>
-  </joint>
   <!-- base_link → camera_link -->
   <joint name="base_to_camera" type="fixed">
